File: V2.kicad_pcb (KiCad board)
At the start: 2 copper layers, 50 x 65 mm, 27 parts, among them J1 RFID_Conn, J2 Connections, J3 IR_SENSOR, J4 SERVO, J5 GND, J6 5V, J7 PWR

Commit message: Hardware design files in KiCad
Routing:
- net KEY_PIN: track 44.2 -> 35.5 mm
Other:
- board size 50 x 65 mm -> 49.9 x 64 mm
Changed lines of the file:
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@@
 			(pintype "passive")
 		)
-		(pad "2" thru_hole oval
+		(pad "2" thru_hole circle
 			(at 5.08 0 180)
-			(size 1.4 1.4)
-			(drill 0.7)
+			(size 2 2)
+			(drill 1)
 			(layers "*.Cu" "*.Mask")
 			(remove_unused_layers no)
@@
 		(pad "1" thru_hole circle
 			(at 0 0 270)
-			(size 1.4 1.4)
-			(drill 0.7)
+			(size 2 2)
+			(drill 1)
 			(layers "*.Cu" "*.Mask")
 			(remove_unused_layers no)
@@
 			(pintype "passive")
 		)
-		(pad "2" thru_hole oval
+		(pad "2" thru_hole circle
 			(at 5.08 0 270)
-			(size 1.4 1.4)
-			(drill 0.7)
+			(size 2 2)
+			(drill 1)
 			(layers "*.Cu" "*.Mask")
 			(remove_unused_layers no)
@@
 	)
 	(gr_line
-		(start 99 79)
-		(end 149 79)
+		(start 99.1 80.01)
+		(end 149 80)
 		(stroke
 			(width 0.05)
@@
 	)
 	(gr_line
-		(start 149 79)
+		(start 149 80)
 		(end 149.03 143.99)
 		(stroke
@@
 	(gr_line
 		(start 99.4 144)
-		(end 99 79)
+		(end 99.1 80.01)
 		(stroke
 			(width 0.05)
@@
 		(layer "Edge.Cuts")
 		(pts
+			(xy 99.4 144) (xy 149.03 143.99)
+		)
+		(height 3.939043)
+		(gr_text "49.6300 mm"
+			(at 124.215562 146.784043 0.01154458568)
+			(layer "Edge.Cuts")
+			(effects
+				(font
+					(size 1 1)
+					(thickness 0.15)
+				)
+			)
+		)
+		(format
+			(prefix "")
+			(suffix "")
+			(units 3)
+			(units_format 1)
+			(precision 4)
+		)
+		(style
+			(thickness 0.05)
+			(arrow_length 1.27)
+			(text_position_mode 0)
+			(extension_height 0.58642)
+			(extension_offset 0.5) keep_text_aligned)
+	)
+	(dimension
+		(type aligned)
+		(layer "Edge.Cuts")
+		(pts
 			(xy 149 79) (xy 124 79)
 		)
@@
 			(extension_offset 0.5) keep_text_aligned)
 	)
+	(dimension
+		(type aligned)
+		(layer "Edge.Cuts")
+		(pts
+			(xy 149 80) (xy 149.03 143.99)
+		)
+		(height -6.836634)
+		(gr_text "63.9900 mm"
+			(at 157.001633 111.991256 270.0268616)
+			(layer "Edge.Cuts")
+			(effects
+				(font
+					(size 1 1)
+					(thickness 0.15)
+				)
+			)
+		)
+		(format
+			(prefix "")
+			(suffix "")
+			(units 3)
+			(units_format 1)
+			(precision 4)
+		)
+		(style
+			(thickness 0.05)
+			(arrow_length 1.27)
+			(text_position_mode 0)
+			(extension_height 0.58642)
+			(extension_offset 0.5) keep_text_aligned)
+	)
 	(segment
 		(start 135.31 125.67)
@@
 	)
 	(segment
-		(start 134.49 123.53)
-		(end 130.07 123.53)
-		(width 1.2)
-		(layer "F.Cu")
-		(net 1)
-	)
-	(segment
-		(start 135.32 124.36)
-		(end 134.96 124)
+		(start 134.04 123.66)
+		(end 135.32 124.94)
 		(width 1.2)
 		(layer "F.Cu")
@@
 	)
 	(segment
-		(start 134.96 124)
-		(end 134.02 124)
-		(width 1.2)
-		(layer "F.Cu")
-		(net 1)
-	)
-	(segment
-		(start 135.32 124.36)
+		(start 135.32 124.94)
 		(end 135.32 125.66)
 		(width 1.2)
@@
 	)
 	(segment
-		(start 134.49 123.53)
-		(end 135.32 124.36)
-		(width 1.2)
-		(layer "F.Cu")
-		(net 1)
-	)
-	(segment
 		(start 134.2 90.46127)
 		(end 139.39 85.27127)
@@
 	)
 	(segment
-		(start 134.02 124)
-		(end 134.49 123.53)
-		(width 1.2)
-		(layer "F.Cu")
-		(net 1)
-	)
-	(segment
-		(start 133.3 124)
-		(end 134.02 124)
-		(width 1.2)
-		(layer "F.Cu")
-		(net 1)
-	)
-	(segment
 		(start 135.32 125.66)
 		(end 135.31 125.67)
@@
 	)
 	(segment
-		(start 134.49 123.53)
-		(end 133.77 123.53)
-		(width 1.2)
-		(layer "F.Cu")
-		(net 1)
-	)
-	(segment
-		(start 129.6 124)
-		(end 133.3 124)
-		(width 1.2)
-		(layer "F.Cu")
-		(net 1)
-	)
-	(segment
-		(start 134.45 109.16)
-		(end 134.2 108.91)
+		(start 130.78 124)
+		(end 129.6 124)
 		(width 1.2)
 		(layer "F.Cu")
@@
 	)
 	(segment
-		(start 133.77 123.53)
-		(end 133.3 124)
+		(start 139.39 85.27127)
+		(end 139.39 83.8)
 		(width 1.2)
 		(layer "F.Cu")
@@
 	)
 	(segment
-		(start 139.39 85.27127)
-		(end 139.39 83.8)
+		(start 131.12 123.66)
+		(end 130.78 124)
 		(width 1.2)
 		(layer "F.Cu")
@@
 	)
 	(segment
-		(start 130.07 123.53)
-		(end 129.6 124)
+		(start 134.04 123.66)
+		(end 131.12 123.66)
 		(width 1.2)
 		(layer "F.Cu")
@@
 	)
 	(via
-		(at 134.49 123.53)
-		(size 1.7)
+		(at 134.04 123.66)
+		(size 2)
 		(drill 1)
 		(layers "F.Cu" "B.Cu")
@@
 	)
 	(via
-		(at 134.45 109.16)
-		(size 1.7)
+		(at 134.21 108.94)
+		(size 2)
 		(drill 1)
 		(layers "F.Cu" "B.Cu")
@@
 	(via
 		(at 116.62 138.9)
-		(size 1.7)
+		(size 2)
 		(drill 1)
 		(layers "F.Cu" "B.Cu")
@@
 	(via
 		(at 125.81 138.92)
-		(size 1.7)
+		(size 2)
 		(drill 1)
 		(layers "F.Cu" "B.Cu")
@@
 	)
 	(via
-		(at 142.18 124.21)
-		(size 1.7)
+		(at 141.83 124)
+		(size 2)
 		(drill 1)
 		(layers "F.Cu" "B.Cu")
@@
 	(via
 		(at 141.91 118.64)
-		(size 1.7)
+		(size 2)
 		(drill 1)
 		(layers "F.Cu" "B.Cu")
@@
 	(via
 		(at 126.35 102.62)
-		(size 1.7)
+		(size 2)
 		(drill 1)
 		(layers "F.Cu" "B.Cu")
@@
 	(via
 		(at 116.48 130.09)
-		(size 1.7)
+		(size 2)
 		(drill 1)
 		(layers "F.Cu" "B.Cu")
@@
 	(via
 		(at 125.87 130.13)
-		(size 1.7)
+		(size 2)
 		(drill 1)
 		(layers "F.Cu" "B.Cu")
@@
 	(via
 		(at 118.28 140.87)
-		(size 1.7)
+		(size 2)
 		(drill 1)
 		(layers "F.Cu" "B.Cu")
@@
 	(via
 		(at 127.051482 140.87)
-		(size 1.7)
+		(size 2)
 		(drill 1)
 		(layers "F.Cu" "B.Cu")
@@
 	(via
 		(at 100.75 134.2)
-		(size 1.7)
+		(size 2)
 		(drill 1)
 		(layers "F.Cu" "B.Cu")
@@
 	(via
 		(at 122.3 134.21322)
-		(size 1.7)
+		(size 2)
 		(drill 1)
 		(layers "F.Cu" "B.Cu")
@@
 	)
 	(segment
-		(start 128.516094 134.16)
-		(end 126.206094 136.47)
+		(start 105.62 133.82)
+		(end 105.62 134.83)
 		(width 1.2)
 		(layer "F.Cu")
@@
 	)
 	(segment
-		(start 105.62 133.82)
-		(end 105.62 134.83)
+		(start 124.154822 136.47)
+		(end 123.904822 136.72)
 		(width 1.2)
 		(layer "F.Cu")
@@
 	)
 	(segment
-		(start 124.154822 136.47)
-		(end 123.904822 136.72)
+		(start 128.516094 134.16)
+		(end 125.856094 136.82)
 		(width 1.2)
 		(layer "F.Cu")
@@
 	)
 	(segment
-		(start 126.206094 136.47)
-		(end 124.154822 136.47)
+		(start 129.6 134.16)
+		(end 128.516094 134.16)
 		(width 1.2)
 		(layer "F.Cu")
@@
 	)
 	(segment
+		(start 124.004822 136.82)
+		(end 123.904822 136.72)
+		(width 1.2)
+		(layer "F.Cu")
+		(net 19)
+	)
+	(segment
 		(start 109.52 83.76)
 		(end 109.52 92.45873)
@@
 	)
 	(segment
-		(start 129.6 134.16)
-		(end 128.516094 134.16)
+		(start 125.856094 136.82)
+		(end 124.004822 136.82)
 		(width 1.2)
 		(layer "F.Cu")
@@
 	(via
 		(at 107.53 136.74)
-		(size 1.7)
+		(size 2)
 		(drill 1)
 		(layers "F.Cu" "B.Cu")
@@
 	(via
 		(at 123.904822 136.72)
-		(size 1.7)
+		(size 2)
 		(drill 1)
 		(layers "F.Cu" "B.Cu")
@@
 	(via
 		(at 123.55 131.82)
-		(size 1.7)
+		(size 2)
 		(drill 1)
 		(layers "F.Cu" "B.Cu")

Commit message: Add BOM
Parts:
- removed A1: Arduino_Nano_v3.x, Module:Arduino_Nano
- removed J4: SERVO, Connector_PinHeader_2.54mm:PinHeader_1x01_P2.54mm_Vertical
- removed kibuzzard-672CC104: G***, kibuzzard-672CC104
- removed kibuzzard-672CC10E: G***, kibuzzard-672CC10E
- removed kibuzzard-672CC151: G***, kibuzzard-672CC151
- removed kibuzzard-672CC18C: G***, kibuzzard-672CC18C
- removed kibuzzard-672CC227: G***, kibuzzard-672CC227
- removed kibuzzard-672CC267: G***, kibuzzard-672CC267
- removed kibuzzard-672CC2CC: G***, kibuzzard-672CC2CC
- removed kibuzzard-672CC2F8: G***, kibuzzard-672CC2F8
- removed kibuzzard-672CC32C: G***, kibuzzard-672CC32C
- removed kibuzzard-672CC353: G***, kibuzzard-672CC353
- removed kibuzzard-672CC370: G***, kibuzzard-672CC370
- removed kibuzzard-672CC3B5: G***, kibuzzard-672CC3B5
- removed kibuzzard-672CC427: G***, kibuzzard-672CC427
- removed kibuzzard-672CC489: G***, kibuzzard-672CC489
- added C1: 100nF, Capacitor_THT:CP_Radial_D5.0mm_P2.50mm, F.Cu at (196.8, 80.6)
- added C2: 100nF, Capacitor_THT:CP_Radial_D5.0mm_P2.50mm, F.Cu at (196.8, 83.7)
- added C3: 22pF, Capacitor_THT:CP_Radial_D5.0mm_P2.50mm, F.Cu at (168.9, 81.1)
- added C4: 22pF, Capacitor_THT:CP_Radial_D5.0mm_P2.50mm, F.Cu at (171.3, 87.7)
- added C5: 100nF, Capacitor_THT:CP_Radial_D5.0mm_P2.50mm, F.Cu at (179.8, 76.5)
- added D3: LED, LED_SMD:LED_0805_2012Metric, F.Cu at (165.7, 64.1)
- added D4: LED, LED_SMD:LED_0805_2012Metric, F.Cu at (165.7, 61.1)
- added D5: LED, LED_SMD:LED_0805_2012Metric, F.Cu at (165.7, 58.0)
- added G***: LOGO, LOGO, F.Cu at (174.7, 60.1)
- added R3: 1M, Resistor_THT:R_Axial_DIN0207_L6.3mm_D2.5mm_P7.62mm_Horizontal, F.Cu at (180.7, 80.7)
- added R4: 1K, Resistor_THT:R_Axial_DIN0207_L6.3mm_D2.5mm_P7.62mm_Horizontal, F.Cu at (194.9, 67.7)
- added R5: 1k, Resistor_SMD:R_0805_2012Metric, F.Cu at (162.2, 64.1)
- added R6: 1k, Resistor_SMD:R_0805_2012Metric, F.Cu at (162.2, 61.1)
- added R7: 1k, Resistor_SMD:R_0805_2012Metric, F.Cu at (162.2, 58.0)
- added SW1: SW_Push, Button_Switch_SMD:SW_SPST_B3U-1000P-B, F.Cu at (198.2, 72.1)
- added U1: ATmega328P-PU, Package_DIP:DIP-28_W7.62mm_Socket_LongPads, F.Cu at (184.2, 62.8)
- added Y1: 16 Mhz, Crystal:Crystal_HC49-4H_Vertical, F.Cu at (175.7, 82.0)
- added kibuzzard-674B2007: G***, kibuzzard-674B2007, F.Cu at (195.5, 63.6)
- added kibuzzard-674B20BC: G***, kibuzzard-674B20BC, F.Cu at (165.1, 54.0)
- added kibuzzard-674B20CA: G***, kibuzzard-674B20CA, F.Cu at (167.9, 54.0)
- added kibuzzard-674B218C: G***, kibuzzard-674B218C, F.Cu at (191.7, 48.4)
- added kibuzzard-674B2203: G***, kibuzzard-674B2203, F.Cu at (191.7, 45.6)
- added kibuzzard-674B266F: G***, kibuzzard-674B266F, F.Cu at (171.0, 54.0)
- added kibuzzard-674B267A: G***, kibuzzard-674B267A, F.Cu at (162.1, 54.0)
- added kibuzzard-674B2C7F: G***, kibuzzard-674B2C7F, F.Cu at (164.5, 48.2)
- added kibuzzard-674B2CD4: G***, kibuzzard-674B2CD4, F.Cu at (195.4, 54.2)
- added kibuzzard-674B2E7C: G***, kibuzzard-674B2E7C, F.Cu at (171.1, 48.2)
- added kibuzzard-674B2E9A: G***, kibuzzard-674B2E9A, F.Cu at (174.2, 48.2)
- added kibuzzard-674B2EE4: G***, kibuzzard-674B2EE4, F.Cu at (177.1, 48.2)
- added kibuzzard-674B2EF3: G***, kibuzzard-674B2EF3, F.Cu at (180.0, 48.2)
- added kibuzzard-674B2F0D: G***, kibuzzard-674B2F0D, F.Cu at (183.8, 48.2)
- added kibuzzard-674B2F1D: G***, kibuzzard-674B2F1D, F.Cu at (186.7, 48.2)
- added kibuzzard-674B2F69: G***, kibuzzard-674B2F69, F.Cu at (189.4, 48.2)
- added kibuzzard-674B41C3: G***, kibuzzard-674B41C3, F.Cu at (182.0, 62.8)
- J3: value IR_SENSOR -> IR_SENSOR n SERVO; footprint Connector_PinHeader_2.54mm:PinHeader_1x01_P2.54mm_Vertical -> Connector_PinHeader_2.54mm:PinHeader_1x02_P2.54mm_Vertical
- R1, R2: footprint Resistor_THT:R_Axial_DIN0204_L3.6mm_D1.6mm_P5.08mm_Horizontal -> Resistor_THT:R_Axial_DIN0207_L6.3mm_D2.5mm_P7.62mm_Horizontal
- moved BZ1 84.6 mm to (191.1, 58.4), turned to 90 degrees
- moved J5 80.8 mm to (197.9, 56.1)
- moved J1 77.0 mm to (171.4, 45.8)
- moved J3 72.8 mm to (194.2, 46.0)
- moved D2 70.9 mm to (179.3, 67.9)
- moved R1 63.0 mm to (180.7, 92.1)
- moved J7 62.3 mm to (197.7, 62.2), turned to 0 degrees
- moved J6 61.4 mm to (162.1, 46.0), turned to 90 degrees
- moved R2 55.2 mm to (180.7, 95.3), turned to 180 degrees
- moved D1 53.6 mm to (166.9, 95.0)
- moved J2 39.7 mm to (162.8, 51.8)
Connections:
- J7 pad 1: VIN -> 5V
Routing:
- net GND: track 99.0 -> 50.7 mm, vias 1 -> 3
- net RFID_MISO: track 66.2 -> 114.1 mm, vias 2 -> 1
- net RFID_MOSI: track 62.6 -> 106.1 mm, vias 2 -> 1
- net RFID_RST: track 57.4 -> 98.9 mm
- net RFID_SDA(SS): track 60.4 -> 96.4 mm, vias 2 -> 1
- net KEY_PIN: track 35.5 -> 68.0 mm, vias 2 -> 0
- net RFID_SCK: track 90.3 -> 116.9 mm, vias 2 -> 1
- net 5V: track 121.1 -> 95.1 mm
- net IR_SENSOR: track 32.1 -> 54.5 mm
- net /D0: track 0.00 -> 19.3 mm
- net /D1: track 0.00 -> 19.1 mm
- net /DTR: track 0.00 -> 18.3 mm, vias 0 -> 2
- net LCK_RETRACTED: track 42.9 -> 58.9 mm, vias 0 -> 1
- net Net-(U1-XTAL2/PB7): track 0.00 -> 14.9 mm
- net Green_LED: track 3.51 -> 18.3 mm
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- added copper zone on F.Cu, net 5V
- added copper zone on B.Cu, net GND
Other:
- board size 49.9 x 64 mm -> 40 x 60 mm
