File: V2.kicad_sch (KiCad schematic)
At the start: 13 parts, among them J1 RFID_Conn, J2 Connections, J3 IR_SENSOR, J4 SERVO, J5 GND, J6 5V, J7 PWR

Commit message: Add BOM
Parts:
- removed A1: Arduino_Nano_v3.x, Module:Arduino_Nano, symbol MCU_Module:Arduino_Nano_v3.x
- removed J4: SERVO, Connector_PinHeader_2.54mm:PinHeader_1x01_P2.54mm_Vertical, symbol Connector:Conn_01x01_Pin
- added C1, C2, C5: 100nF, Capacitor_THT:CP_Radial_D5.0mm_P2.50mm, symbol stormduino-Rev2-rescue:C-Device
- added C3, C4: 22pF, Capacitor_THT:CP_Radial_D5.0mm_P2.50mm, symbol stormduino-Rev2-rescue:C-Device
- added D3, D4, D5: LED, LED_SMD:LED_0805_2012Metric, symbol stormduino-Rev2-rescue:LED-Device
- added R3: 1M, Resistor_THT:R_Axial_DIN0207_L6.3mm_D2.5mm_P7.62mm_Horizontal, symbol stormduino-Rev2-rescue:R-Device
- added R4: 1K, Resistor_THT:R_Axial_DIN0207_L6.3mm_D2.5mm_P7.62mm_Horizontal, symbol stormduino-Rev2-rescue:R-Device
- added R5, R6, R7: 1k, Resistor_SMD:R_0805_2012Metric, symbol stormduino-Rev2-rescue:R-Device
- added SW1: SW_Push, Button_Switch_SMD:SW_SPST_B3U-1000P-B, symbol stormduino-Rev2-rescue:SW_Push-Switch
- added U1: ATmega328P-PU, Package_DIP:DIP-28_W7.62mm_Socket_LongPads, symbol MCU_Microchip_ATmega:ATmega328P-P
- added Y1: 16 Mhz, Crystal:Crystal_HC49-4H_Vertical, symbol stormduino-Rev2-rescue:Crystal-Device
- J3: value IR_SENSOR -> IR_SENSOR n SERVO; footprint Connector_PinHeader_2.54mm:PinHeader_1x01_P2.54mm_Vertical -> Connector_PinHeader_2.54mm:PinHeader_1x02_P2.54mm_Vertical; symbol Connector:Conn_01x01_Pin -> Connector:Conn_01x02_Pin
- R1, R2: footprint Resistor_THT:R_Axial_DIN0204_L3.6mm_D1.6mm_P5.08mm_Horizontal -> Resistor_THT:R_Axial_DIN0207_L6.3mm_D2.5mm_P7.62mm_Horizontal
Connections:
- net VIN is gone; now on net +5V: J7.1 (Pin_1)
- net BUZZER_PIN: now also U1.28 (PC5)
- net EXT_ALARM: now also U1.26 (PC3)
- net GND: now also C1.2, C2.2, C3.1, C4.2, C5.2, D5.1 (K), SW1.1, U1.22 (GND), U1.8 (GND)
- net Green_LED: now also U1.14 (PB0)
- net IR_SENSOR: now also U1.12 (PD6)
- net KEY_PIN: now also U1.13 (PD7)
- net LCK_EXTENDED: now also U1.6 (PD4)
- net LCK_RETRACTED: now also U1.11 (PD5)
- net RFID_MISO: now also U1.18 (PB4)
- net RFID_MOSI: now also U1.17 (PB3)
- net RFID_RST: now also U1.15 (PB1)
- net RFID_SCK: now also U1.19 (PB5)
- net RFID_SDA(SS): now also U1.16 (PB2)
- net Red_LED: now also U1.4 (PD2)
- net SERVO_PIN: now also J3.2 (Pin_2), U1.5 (PD3)
- net 5V renamed +5V
- net +5V: now also C2.1, C5.1, R4.2, R5.2, R6.1, R7.1, U1.20 (AVCC), U1.7 (VCC)
- new net: D4.2 (A), R6.2
- new net: D5.2 (A), R7.2
- new net: C4.1, R3.2, U1.10 (XTAL2/PB7), Y1.2
- new net: C3.2, R3.1, U1.9 (XTAL1/PB6), Y1.1
- new net: D3.2 (A), R5.1
- new net A0: U1.23 (PC0)
- new net A1: U1.24 (PC1)
- new net A2: U1.25 (PC2)
- new net A4: U1.27 (PC4)
- new net AREF: C1.1, U1.21 (AREF)
- new net D0: D4.1 (K), U1.2 (PD0)
- new net D1: D3.1 (K), U1.3 (PD1)
- new net DTR: R4.1, SW1.2, U1.1 (~{RESET}/PC6)
- no-connect marks 12 -> 6
Other:
- note added: "LEDS"
- note added: "RESET SWITCH"
- company: (none) -> Karama Tech
- moved on the sheet: BZ1, D1, D2, J1, J2, J5, J6, J7, R1, R2
